File: Hardware/Eagle/LVMi Pressure Sensor/2022-07-29 LVMi Pressure Sensor - 1624.brd (EAGLE design)
At the start: 53.3 x 94 mm, 26 parts, among them J1 POWER_JACKPJ-102AH, SW1 SWITCH-RA-800BWSP9SM6RE, U1 ATTINY1624-SSU, U2 Sensiron SDP800

Commit message: WIP
Parts:
- added C7, C8: 0.1uF, AUmlib:C0805
- added PS1: OKI-78SR-5/1.5-W36-C, AUmlib:CONV_OKI-78SR-5/1.5-W36-C
- added R5: 10K, AUmlib:R0805
- added TP2: +5V, AUmlib:TP5000-TESTPOINT-RED
- added U3: SN74LV1T34DBVR, AUmlib:SOT95P280X145-5N
- added U5: TXB0102DCURVSSOP8, AUmlib:GHI-IC_VSSOP8(TI)
- C1: value 0.1uF -> 10uF 50V; device AUmlib:C0805 -> AUmlib:C1210
- C2: value 10uF 50V -> 0.1uF; device AUmlib:C1210 -> AUmlib:C0805
- R3: value 270K -> (none)
- moved C1 33.1 mm to (15.2, 5.08), flipped to the bottom
- moved C2 32.2 mm to (40.0, 29.8), turned to 90 degrees
- moved TP3 17.9 mm to (9.53, 20.3)
- moved C6 7.10 mm to (32.4, 20.3)
- moved R1 3.81 mm to (31.8, 73.7)
- moved R2 3.81 mm to (27.9, 73.7)
- moved J1 3.70 mm to (6.35, 9.53), turned to 180 degrees
- moved TP1 3.26 mm to (26.0, 6.35)
- moved LS1 1.66 mm to (48.9, 38.7)
- moved D1 0.63 mm to (16.5, 12.1), flipped to the bottom, turned to 0 degrees
- renumbered U1 to U4
Connections:
- new net +5V: C2.1, C8.2, JP1.2, LCD1.3, PS1.3, R1.2, R2.2, TP2.P$1, U2.VDD, U4.1, U5.7
- new net /RST: J2./RST, U3.4
- new net OE: R5.1, U5.6
- new net XP-RX: J2.RX, U5.4
- new net XP-TX: J2.TX, U5.5
- net +3.3V: now also C7.2, R5.2, U3.5, U5.3; no longer C1.1, JP1.2, LCD1.2, LCD1.3, R1.2, R2.2, U2.VDD, U4.1
- net GND: now also C7.1, C8.1, PS1.2, U3.3, U5.2
- net MCU-RX: now also U5.8; no longer J2.TX
- net MCU-TX: now also U5.1; no longer J2.RX
- net SCL: now also R2.1; no longer R1.1
- net SDA: now also R1.1; no longer R2.1
- net VIN: now also C1.1, PS1.1; no longer C2.1
- net XPORT/RST: now also U3.2; no longer J2./RST
Routing:
- net +5V: track 0.00 -> 139.4 mm, vias 0 -> 2
- net +3.3V: track 143.8 -> 55.1 mm, vias 4 -> 2
- net XP-RX: track 0.00 -> 54.9 mm
- net MCU-TX: track 70.7 -> 33.7 mm
- net XP-TX: track 0.00 -> 33.3 mm
- net MCU-RX: track 56.7 -> 27.3 mm
- net /RST: track 0.00 -> 25.1 mm
- net XPORT/RST: track 34.9 -> 21.1 mm
- net VIN: track 10.5 -> 19.3 mm, vias 0 -> 1
- net OE: track 0.00 -> 5.62 mm
- net VSUP: track 4.55 -> 8.47 mm
- net BEEP: track 15.5 -> 17.3 mm
- net GND: track 19.5 -> 20.6 mm, vias 5 -> 9
Other:
- board text added: "2022-07-28 LVMi Dewar Air Sensor"
- board text removed: "2022-07-29 LVMi Dewar Air Sensor"
- board text removed: "UPDI"
